File: Hardware/Proiect_v132.brd (EAGLE design)
At the start: 170.2 x 111.2 mm, 103 parts, among them IC1 BD5229G-TR, IC4 XC6220A331MR-GIC4, J1 FH34SRJ-24S-0.5SH_99_, J2 SAMACSYS_PARTS_USB4110-GF-A, J3 QWIIC_RIGHT_ANGLE, J4 112A-TAAR-R03_ATTEND, Q1 20V/4.2A/52mΩ/1.4W, Q2 20V/4.2A/52mΩ/1.4W, Q3 SI1308EDL-T1-GE3, U1 W25Q512JVEIQ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

Commit message: am rezolvat issue-urile si am adaugat fisierele
Parts:
- moved J4 11.7 mm to (6.59, 94.7), turned to 270 degrees
- moved TP13 2.42 mm to (99.7, 11.9)
Routing:
- net GND: track 761.8 -> 699.4 mm
- net SCK: track 147.4 -> 167.9 mm, vias 6 -> 7
- net MISO: track 63.1 -> 75.5 mm, vias 3 -> 4
- net MOSI: track 137.4 -> 142.9 mm, vias 5 -> 7
- net 3V3: track 454.9 -> 458.9 mm, vias 7 -> 8
- net SS_SD: track 41.3 -> 45.3 mm
- net EPD_3V3_C: track 123.9 -> 126.5 mm
